Commit message: Added new package tiago_pro_base_anchor which helps to hold/release tiago robot in gazebo and Updated README

File: tiago_pro/share/omni_base_description/urdf/base/base.urdf.xacro (robot description, xacro)
@@ -72,4 +72,10 @@
       <parent link="${name}_footprint"/>
     </joint>
+    <!-- Fixed joint to attach robot to the world -->
+    <!-- <joint name="${name}_world_fixed" type="fixed">
+      <parent link="world"/>
+      <child link="${name}_footprint"/>
+      <origin xyz="0 0 0" rpy="0 0 0"/>
+    </joint> -->
     <!-- Docking link -->
     <link name="${name}_dock_link">

Commit message: Updated pick_cube_node in cartesian_mover package

File: tiago_pro/share/omni_base_description/urdf/base/base.urdf.xacro (robot description, xacro)
@@ -72,10 +72,4 @@
       <parent link="${name}_footprint"/>
     </joint>
-    <!-- Fixed joint to attach robot to the world -->
-    <!-- <joint name="${name}_world_fixed" type="fixed">
-      <parent link="world"/>
-      <child link="${name}_footprint"/>
-      <origin xyz="0 0 0" rpy="0 0 0"/>
-    </joint> -->
     <!-- Docking link -->
     <link name="${name}_dock_link">
